File: PushPull-fingers/fingers.sch (KiCad schematic (older format))
At the start: 2 parts, among them P1 CONN_01X07, U1 fingerBoard

Commit message: production pcb kicad files and gerbers
Parts:
- removed P1: CONN_01X07, Connectors_Molex:Connector_Molex_PicoBlade_53398-0771, symbol CONN_01X07
- removed U1: fingerBoard, PushPull:pushPullFingersPad, symbol fingerBoard
- added P?: CapFingers, symbol CONN_01X08
- added P?: CONN_01X08, symbol CONN_01X08
Connections:
- net GND: now also P?.2 (P2), P?.2 (P2), P?.4 (P4), P?.4 (P4), P?.6 (P6), P?.6 (P6), P?.8 (P8), P?.8 (P8)
- new net: P?.1 (P1), P?.1 (P1)
- new net: P?.3 (P3), P?.3 (P3)
- new net: P?.5 (P5), P?.5 (P5)
- new net: P?.7 (P7), P?.7 (P7)
Changed lines of the file:
@@
 LIBS:memory
 LIBS:xilinx
+LIBS:special
 LIBS:microcontrollers
 LIBS:dsp
@@
 LIBS:contrib
 LIBS:valves
-LIBS:pushPullComponents
 LIBS:fingers-cache
 EELAYER 25 0
@@
 Comment4 ""
 $EndDescr
-$Comp
-L fingerBoard U1
-U 1 1 5550B8F6
-P 6050 3500
-F 0 "U1" H 6050 4050 60  0000 C CNN
-F 1 "fingerBoard" H 6050 3550 60  0000 C CNN
-F 2 "PushPull:pushPullFingersPad" H 5750 3500 60  0001 C CNN
-F 3 "" H 5750 3500 60  0000 C CNN
-	1    6050 3500
-	1    0    0    -1
-$EndComp
-$Comp
-L CONN_01X07 P1
-U 1 1 5550B930
-P 3900 3250
-F 0 "P1" H 3900 3700 50  0000 C CNN
-F 1 "CONN_01X07" V 4000 3250 50  0000 C CNN
-F 2 "Connectors_Molex:Connector_Molex_PicoBlade_53398-0771" H 3900 3250 60  0001 C CNN
-F 3 "" H 3900 3250 60  0000 C CNN
-	1    3900 3250
-	-1   0    0    -1
-$EndComp
 Wire Wire Line
 	4100 2950 5650 2950
 Wire Wire Line
-	5650 2950 5650 3050
-Wire Wire Line
 	4100 3150 5650 3150
 Wire Wire Line
-	4100 3350 5050 3350
+	4100 3350 5650 3350
 Wire Wire Line
-	5050 3350 5050 3250
-Wire Wire Line
-	5050 3250 5650 3250
-Wire Wire Line
-	4100 3550 5300 3550
-Wire Wire Line
-	5300 3550 5300 3350
-Wire Wire Line
-	5300 3350 5650 3350
+	4100 3550 5650 3550
 $Comp
-L GND #PWR01
+L GND #PWR1
 U 1 1 5550B9DB
 P 4300 2700
-F 0 "#PWR01" H 4300 2450 50  0001 C CNN
+F 0 "#PWR1" H 4300 2450 50  0001 C CNN
 F 1 "GND" H 4300 2550 50  0000 C CNN
 F 2 "" H 4300 2700 60  0000 C CNN
@@
 $EndComp
 Wire Wire Line
-	4300 2700 4300 3450
+	4300 2700 4300 3650
 Wire Wire Line
-	4300 3450 4100 3450
+	4100 3450 5650 3450
 Wire Wire Line
-	4100 3250 4300 3250
+	4100 3250 5650 3250
 Connection ~ 4300 3250
 Wire Wire Line
-	4100 3050 4300 3050
+	4100 3050 5650 3050
 Connection ~ 4300 3050
+Connection ~ 4300 2800
+Connection ~ 4300 3450
+$Comp
+L CONN_01X08 P?
+U 1 1 5564A168
+P 3900 3300
+F 0 "P?" H 3900 3750 50  0000 C CNN
+F 1 "CapFingers" V 4000 3300 50  0000 C CNN
+F 2 "" H 3900 3300 60  0000 C CNN
+F 3 "" H 3900 3300 60  0000 C CNN
+	1    3900 3300
+	-1   0    0    -1
+$EndComp
 Wire Wire Line
-	4300 2800 6600 2800
-Wire Wire Line
-	6600 2800 6600 3350
-Wire Wire Line
-	6600 3350 6450 3350
-Connection ~ 4300 2800
-Wire Wire Line
-	6450 3250 6600 3250
-Connection ~ 6600 3250
-Wire Wire Line
-	6450 3150 6600 3150
-Connection ~ 6600 3150
-Wire Wire Line
-	6450 3050 6600 3050
-Connection ~ 6600 3050
+	4100 3650 5650 3650
+$Comp
+L CONN_01X08 P?
+U 1 1 5564A223
+P 5850 3300
+F 0 "P?" H 5850 3750 50  0000 C CNN
+F 1 "CONN_01X08" V 5950 3300 50  0000 C CNN
+F 2 "" H 5850 3300 60  0000 C CNN
+F 3 "" H 5850 3300 60  0000 C CNN
+	1    5850 3300
+	1    0    0    -1
+$EndComp
+Connection ~ 4300 3650
 $EndSCHEMATC
