File: PushPull-main/mainPCB.sch (KiCad schematic (older format))
At the start: 16 parts

Commit message: production pcb kicad files and gerbers
Parts:
- removed P?: CAP Conn, symbol CONN_01X11
- added C1, C2, C3, C4: 1µ, symbol C
- added C5: 470µ, symbol CP
- added P2: CapFingers, symbol CONN_01X08
- added P5: CapThumb, symbol CONN_01X04
- added R7: 100, symbol R
- P1: renamed from P?; value POWER Conn -> Battery 3.7V
- P3: renamed from P?; value TO LOWER -> to lower
- P4: renamed from P?; value Debug Conn -> debug port
- R1: renamed from R?; value R -> Rcap1
- R2: renamed from R?; value R -> Rcap2
- R3: renamed from R?; value R -> Rcap3
- R4: renamed from R?; value R -> Rcap4
- R5: renamed from R?; value R -> Rcap5
- R6: renamed from R?; value R -> Rcap6
- U1, U2, U3, U4: renamed from U?; value NEOPixel_BBFriend -> NEOPixel
- U5: renamed from U?; value X-OSC_v1.6 -> X-OSC v1.6
- U6: renamed from U?; value CY8CKIT-049-42XX -> Cypress CY8CKIT-049-42XX
Connections:
- net GND: now also P4.4 (P4), C1.2, C2.2, C3.2, C4.2, C5.2, P2.2 (P2), P2.4 (P4), P2.6 (P6), P2.8 (P8), P5.2 (P2), P5.4 (P4); no longer P4.2 (P2)
- net VDD: now also U1.1 (VDD), U2.1 (VDD), U3.1 (VDD), U4.1 (VDD), C1.1, C2.1, C3.1, C4.1, C5.1
- net at U6.18 (P3.2_SWDIO): now also P4.1 (P1); no longer P4.5 (P5)
- net at U6.19 (P3.3_SWDCLK): now also P4.2 (P2); no longer P4.4 (P4)
- net at U6.22 (P4.VDD): now also P4.5 (P5); no longer P4.1 (P1)
- net at U6.30 (0.3): now also R3.1; no longer R1.1
- net at U6.39 (1.4): now also R1.1; no longer R3.1
- net at U5.19 (Out_01): now also R7.2; no longer U1.3 (DIN)
- net at R3.2: now also P2.5 (P5)
- net at R4.2: now also P2.7 (P7)
- net at R5.2: now also P5.1 (P1)
- net at R6.2: now also P5.3 (P3)
- net at R2.2: now also P2.3 (P3)
- net at R1.2: now also P2.1 (P1)
- new net: R7.1, U1.3 (DIN)
