File: PushPull-thumb/thumb.kicad_pcb (KiCad board)
At the start: 2 copper layers, 2 parts, among them P1 Connector, P2 CapSense

Commit message: production pcb kicad files and gerbers
Parts:
- P1: value Connector -> CapThumb; footprint Connect:GS3 -> Pushpull:4_PIN_MM_conn
- P2: value CapSense -> Thumb; footprint PushPull:pushPullThumbPad-Cu-final -> Pushpull:PushPull_ThumbLogo
- moved P1 8.35 mm to (147.3, 103.5), turned to 0 degrees
Connections:
- P1 pad 3: /antennae -> Net-(P1-Pad3)
- P2 pad 1: /antennae -> Net-(P1-Pad1)
- P2 pad 3: Net-(P1-Pad1) -> Net-(P1-Pad3)
Routing:
- net GND: track 7.33 -> 28.3 mm
- net Net-(P1-Pad3): track 0.00 -> 13.3 mm
- net /antennae: track 6.51 -> 0.00 mm
- added copper zone on B.Cu, net GND
Other:
- board outline added: 26.6 x 28.3 mm
- board text added: "3DMin PushPull Udk Berlin 2015 Thumb PCB rev 01"
