File: PushPull-thumb/thumb.sch (KiCad schematic (older format))
At the start: 2 parts, among them P1 Connector, P2 CapSense

Commit message: production pcb kicad files and gerbers
Parts:
- removed P1: Connector, Connect:GS3, symbol CONN_01X03
- removed P2: CapSense, PushPull:pushPullThumbPad-Cu-final, symbol CONN_01X03
- added P1: Mainboard, symbol CONN_01X04
- added P2: Thumb, symbol CONN_01X04
Connections:
- net GND: now also P1.1 (P1), P1.3 (P3), P2.1 (P1), P2.3 (P3)
- new net: P1.2 (P2), P2.2 (P2)
- new net: P1.4 (P4), P2.4 (P4)
Changed lines of the file:
@@
 LIBS:memory
 LIBS:xilinx
+LIBS:special
 LIBS:microcontrollers
 LIBS:dsp
@@
 $EndDescr
 $Comp
-L CONN_01X03 P1
-U 1 1 554741E4
-P 1500 2700
-F 0 "P1" H 1500 2850 50  0000 C CNN
-F 1 "Connector" V 1600 2700 50  0000 C CNN
-F 2 "Connect:GS3" H 1500 2700 60  0001 C CNN
-F 3 "" H 1500 2700 60  0000 C CNN
-	1    1500 2700
+L GND #PWR01
+U 1 1 554742A4
+P 1850 2400
+F 0 "#PWR01" H 1850 2150 50  0001 C CNN
+F 1 "GND" H 1850 2250 50  0000 C CNN
+F 2 "" H 1850 2400 60  0000 C CNN
+F 3 "" H 1850 2400 60  0000 C CNN
+	1    1850 2400
+	1    0    0    -1
+$EndComp
+$Comp
+L CONN_01X04 P1
+U 1 1 5563B566
+P 1500 2150
+F 0 "P1" H 1500 2400 50  0000 C CNN
+F 1 "Mainboard" V 1600 2150 50  0000 C CNN
+F 2 "" H 1500 2150 60  0000 C CNN
+F 3 "" H 1500 2150 60  0000 C CNN
+	1    1500 2150
 	-1   0    0    1
 $EndComp
-Wire Wire Line
-	1700 2600 3550 2600
-Wire Wire Line
-	1700 2700 3550 2700
-Wire Wire Line
-	3300 2700 3300 3100
 $Comp
-L GND #PWR01
-U 1 1 554742A4
-P 3300 3100
-F 0 "#PWR01" H 3300 2850 50  0001 C CNN
-F 1 "GND" H 3300 2950 50  0000 C CNN
-F 2 "" H 3300 3100 60  0000 C CNN
-F 3 "" H 3300 3100 60  0000 C CNN
-	1    3300 3100
-	1    0    0    -1
-$EndComp
-Text Label 2900 2600 0    60   ~ 0
-antennae
-Connection ~ 3300 2700
-$Comp
-L CONN_01X03 P2
-U 1 1 554B65CC
-P 3750 2700
-F 0 "P2" H 3750 2900 50  0000 C CNN
-F 1 "CapSense" V 3850 2700 50  0000 C CNN
-F 2 "PushPull:pushPullThumbPad-Cu-final" H 3750 2700 60  0001 C CNN
-F 3 "" H 3750 2700 60  0000 C CNN
-	1    3750 2700
-	1    0    0    -1
+L CONN_01X04 P2
+U 1 1 5563B6AE
+P 3000 2150
+F 0 "P2" H 3000 2400 50  0000 C CNN
+F 1 "Thumb" V 3100 2150 50  0000 C CNN
+F 2 "" H 3000 2150 60  0000 C CNN
+F 3 "" H 3000 2150 60  0000 C CNN
+	1    3000 2150
+	1    0    0    1
 $EndComp
 Wire Wire Line
-	1700 2800 3550 2800
+	1700 2300 2800 2300
+Wire Wire Line
+	1700 2100 2800 2100
+Wire Wire Line
+	1700 2200 2800 2200
+Wire Wire Line
+	1700 2000 2800 2000
+Wire Wire Line
+	1850 2100 1850 2400
+Connection ~ 1850 2300
+Connection ~ 1850 2100
 $EndSCHEMATC
