File: PushPull-thumb-left/thumb.sch (KiCad schematic (older format))
At the start: 2 parts, among them P1 Mainboard, P2 Thumb

Commit message: pushpull left hand version cap sense
Parts:
- P1: footprint (none) -> PushPull-footprints:4_PIN_MM_conn
- P2: footprint (none) -> PushPull-footprints:PushPull_ThumbLogo-left
Connections:
- net at P1.1 (P1): now also P2.3 (P3); no longer P2.1 (P1)
- net at P1.3 (P3): now also P2.1 (P1); no longer P2.3 (P3)
Other:
- moved on the sheet: P2
Changed lines of the file:
@@
 F 0 "P1" H 1500 2400 50  0000 C CNN
 F 1 "Mainboard" V 1600 2150 50  0000 C CNN
-F 2 "" H 1500 2150 60  0000 C CNN
+F 2 "PushPull-footprints:4_PIN_MM_conn" H 1500 2150 60  0001 C CNN
 F 3 "" H 1500 2150 60  0000 C CNN
 	1    1500 2150
@@
 L CONN_01X04 P2
 U 1 1 5563B6AE
-P 3000 2150
-F 0 "P2" H 3000 2400 50  0000 C CNN
-F 1 "Thumb" V 3100 2150 50  0000 C CNN
-F 2 "" H 3000 2150 60  0000 C CNN
-F 3 "" H 3000 2150 60  0000 C CNN
-	1    3000 2150
-	1    0    0    1
+P 3000 2250
+F 0 "P2" H 3000 2500 50  0000 C CNN
+F 1 "Thumb" V 3100 2250 50  0000 C CNN
+F 2 "PushPull-footprints:PushPull_ThumbLogo-left" H 3000 2250 60  0001 C CNN
+F 3 "" H 3000 2250 60  0000 C CNN
+	1    3000 2250
+	1    0    0    -1
 $EndComp
 Wire Wire Line
@@
 	1700 2200 2800 2200
 Wire Wire Line
-	1700 2000 2800 2000
+	2550 2000 1700 2000
 Wire Wire Line
 	1850 2000 1850 2400
 Connection ~ 1850 2200
 Connection ~ 1850 2000
+Wire Wire Line
+	2800 2400 2550 2400
+Wire Wire Line
+	2550 2400 2550 2000
 $EndSCHEMATC
