File: PushPull-preAmp/preAmp.kicad_pcb (KiCad board)
At the start: 2 copper layers, 33 parts, among them P1 PWR, P2 OUT, P3 IN, U1 TL072

Commit message: preamp layout single sided
Parts:
- removed C13: 100n, Capacitors_ThroughHole:C_Rect_L4_W2.5_P2.5
- added P4: IN, Pin_Headers:Pin_Header_Straight_1x02, F.Cu at (92.7, 111.8)
- added P5: IN, Pin_Headers:Pin_Header_Straight_1x02, F.Cu at (95.2, 111.8)
- added R15: 22k, Resistors_ThroughHole:Resistor_Horizontal_RM10mm, F.Cu at (85.1, 106.7)
- added R16: 100k, Resistors_ThroughHole:Resistor_Horizontal_RM10mm, F.Cu at (102.9, 106.7)
- added REF**: drill_3.5mm, PushPull-footprints:drill_4mm, F.Cu at (66.0, 69.8)
- added REF**: drill_3.5mm, PushPull-footprints:drill_4mm, F.Cu at (123.2, 110.5)
- added REF**: drill_3.5mm, PushPull-footprints:drill_4mm, F.Cu at (66.0, 110.5)
- added U2: LP2950 3.3V, Discret:TO92, F.Cu at (104.1, 71.1)
- C12: value 220µ -> 4µ7
- C2, C6: value 470n -> 1µ; footprint Capacitors_ThroughHole:C_Rect_L4_W2.5_P2.5 -> Capacitors_ThroughHole:C_Rect_L7_W4.5_P5
- C4, C8: value 4µ7 -> 10µ
- C9: value 4µ7 -> 1µ
- moved P1 135.3 mm to (120.7, 72.4)
- moved C9 129.5 mm to (113.0, 69.8), turned to 270 degrees
- moved C12 113.8 mm to (96.5, 72.4)
- moved R14 110.6 mm to (95.2, 77.5)
- moved C10 83.7 mm to (91.4, 106.7)
- moved C11 82.8 mm to (96.5, 106.7)
- moved RV2 54.6 mm to (108.0, 83.8)
- moved C3 49.8 mm to (67.3, 90.2), turned to 270 degrees
- moved R5 40.7 mm to (77.5, 91.4), turned to 0 degrees
- moved C5 39.8 mm to (120.7, 99.1), turned to 90 degrees
- moved R1 36.1 mm to (69.8, 104.1), turned to 0 degrees
- moved R8 35.3 mm to (118.1, 104.1), turned to 180 degrees
- moved R2 26.7 mm to (90.2, 87.6), turned to 0 degrees
- moved P3 17.0 mm to (77.5, 128.3)
- moved R3 14.9 mm to (77.5, 99.1), turned to 180 degrees
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Connections:
- C10 pad 1: +9V -> +3V3
- C11 pad 1: +9V -> +3V3
- C12 pad 1: +9V -> +3V3
- C4 pad 2: /out1 -> Net-(C4-Pad2)
- C8 pad 2: /out2 -> Net-(C8-Pad2)
- C9 pad 1: +9V -> Net-(C9-Pad1)
- P1 pad 1: +9V -> GND
- P1 pad 2: GND -> Net-(C9-Pad1)
- R1 pad 2: /in1 -> Net-(C2-Pad1)
- R14 pad 1: Net-(C8-Pad1) -> /out2
- R14 pad 2: Net-(R14-Pad2) -> Net-(C8-Pad2)
- R2 pad 2: +9V -> +3V3
- R7 pad 1: Net-(C4-Pad1) -> /out1
- R7 pad 2: Net-(R7-Pad2) -> Net-(C4-Pad2)
- R8 pad 2: /in2 -> Net-(C6-Pad1)
- R9 pad 2: +9V -> +3V3
- RV1 pad 1: Net-(R7-Pad2) -> Net-(R6-Pad1)
- RV1 pad 2: Net-(R7-Pad2) -> Net-(C4-Pad1)
- RV1 pad 3: Net-(R6-Pad1) -> Net-(C4-Pad1)
- RV2 pad 1: Net-(R14-Pad2) -> Net-(R13-Pad1)
- RV2 pad 2: Net-(R14-Pad2) -> Net-(C8-Pad1)
- RV2 pad 3: Net-(R13-Pad1) -> Net-(C8-Pad1)
- U1 pad 1: Net-(R7-Pad2) -> Net-(C4-Pad1)
- U1 pad 7: Net-(R14-Pad2) -> Net-(C8-Pad1)
- U1 pad 8: +9V -> +3V3
Routing:
- net GND: track 44.5 -> 183.8 mm
- net +9V: track 75.5 -> 0.00 mm
- net +3V3: track 0.00 -> 73.9 mm
- net Net-(R5-Pad2): track 47.6 -> 10.2 mm
- net Net-(C8-Pad1): track 0.00 -> 36.3 mm
- net Net-(R7-Pad2): track 26.5 -> 0.00 mm
- net Net-(C4-Pad1): track 5.08 -> 26.5 mm
- net Net-(C5-Pad1): track 5.08 -> 25.7 mm
- net /in1: track 30.6 -> 11.8 mm
- net /in2: track 28.8 -> 11.8 mm
- net Net-(C9-Pad1): track 0.00 -> 15.2 mm
- net Net-(R13-Pad1): track 0.00 -> 12.3 mm
- net /out2: track 0.00 -> 9.72 mm
- net /out1: track 0.00 -> 9.72 mm
- net Net-(C4-Pad2): track 0.00 -> 8.45 mm
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- added copper zone on B.Cu, net GND
Other:
- net class Default: clearance 0.2 -> 0.3; trace_width 0.25 -> 0.4; via_dia 0.6 -> 1.8; via_drill 0.4 -> 0.8
- net class Supply added: clearance 0.3, trace_width 1, via_dia 1.8, via_drill 0.8
- rule trace_clearance: 0.2 -> 0.3

Commit message: preamp layout drills
Parts:
- removed the REF** at (66.0, 69.8)
- removed the REF** at (123.2, 110.5)
- removed the REF** at (66.0, 110.5)
- added REF**: drill_3.5mm, PushPull-footprints:drill_4mm, F.Cu at (77.7, 113.7)
- added REF**: drill_3.5mm, PushPull-footprints:drill_4mm, F.Cu at (110.4, 113.7)
- added REF**: drill_3.5mm, PushPull-footprints:drill_4mm, F.Cu at (77.7, 85.4)
- added REF**: drill_3.5mm, PushPull-footprints:drill_4mm, F.Cu at (110.4, 85.4)
- P1: footprint Pin_Headers:Pin_Header_Straight_1x02 -> Pin_Headers:Pin_Header_Straight_1x03
- P3: value IN -> PWR; footprint Pin_Headers:Pin_Header_Straight_1x02 -> Pin_Headers:Pin_Header_Straight_1x03
- RV1, RV2: footprint Potentiometers:Potentiometer_Trimmer-Piher-PT15-h2-5_vertical -> PushPull-footprints:Trimmer_Dual
- moved P3 68.4 mm to (102.9, 64.8)
- moved P4 22.9 mm to (69.8, 110.5), turned to 0 degrees
- moved P5 22.9 mm to (118.1, 110.5), turned to 0 degrees
- moved R9 21.8 mm to (118.1, 105.4)
- moved RV2 13.5 mm to (118.1, 74.9), turned to 270 degrees
- moved P1 7.73 mm to (121.9, 64.8), turned to 270 degrees
- moved P2 5.08 mm to (87.6, 69.8), turned to 270 degrees
- moved RV1 2.84 mm to (69.8, 85.1), turned to 90 degrees
- moved R8 1.27 mm to (118.1, 102.9)
Connections:
- P2 pad 1: /out1 -> GND
- P2 pad 3: GND -> /out1
- P3 pad 1: /in1 -> GND
- P3 pad 2: /in2 -> Net-(C9-Pad1)
Routing:
- net Net-(C4-Pad1): track 26.5 -> 42.1 mm
- net Net-(R13-Pad1): track 12.3 -> 22.5 mm
- net /TX: track 0.00 -> 8.89 mm
- net Net-(C9-Pad1): track 15.2 -> 22.6 mm
- net /in1: track 11.8 -> 19.0 mm
- net /in2: track 11.8 -> 19.0 mm
- net +3V3: track 73.9 -> 79.2 mm
- net Net-(C8-Pad1): track 36.3 -> 41.0 mm
- net GND: track 183.8 -> 187.5 mm
- net Net-(C5-Pad1): track 25.7 -> 24.4 mm
- net Net-(C6-Pad1): track 18.1 -> 17.6 mm
Other:
- board outline added: 68 x 50 mm
- board text added: "PushPull Pre rev1"
